Commit message: changing find package name

File: urdf/accessories.urdf.xacro (robot description, xacro)
@@ -10,16 +10,16 @@
   -->
   <!-- Macros to generate standoffs for offset payload mounting. -->
-  <xacro:include filename="$(find jackal_velodyne_vlp16_lidar_ros_nav_stack)/urdf/accessories/standoffs.urdf.xacro" />
+  <xacro:include filename="$(find ros_stack_sim_jackal)/urdf/accessories/standoffs.urdf.xacro" />
   <!-- This optional plate mounts both the upgraded GPS and the Velodyne 3D LIDAR. -->
-  <xacro:include filename="$(find jackal_velodyne_vlp16_lidar_ros_nav_stack)/urdf/accessories/bridge_plate.urdf.xacro" />
+  <xacro:include filename="$(find ros_stack_sim_jackal)/urdf/accessories/bridge_plate.urdf.xacro" />
   <!-- 2D Lidars -->
   <xacro:include filename="$(find sick_tim)/urdf/sick_tim.urdf.xacro" />
-  <xacro:include filename="$(find jackal_velodyne_vlp16_lidar_ros_nav_stack)/urdf/accessories/sick_lms1xx.urdf.xacro" />
-  <xacro:include filename="$(find jackal_velodyne_vlp16_lidar_ros_nav_stack)/urdf/accessories/sick_lms1xx_inverted_mount.urdf.xacro" />
-  <xacro:include filename="$(find jackal_velodyne_vlp16_lidar_ros_nav_stack)/urdf/accessories/sick_lms1xx_upright_mount.urdf.xacro" />
-  <xacro:include filename="$(find jackal_velodyne_vlp16_lidar_ros_nav_stack)/urdf/accessories/hokuyo_utm30.urdf.xacro" />
-  <xacro:include filename="$(find jackal_velodyne_vlp16_lidar_ros_nav_stack)/urdf/accessories/hokuyo_ust10.urdf.xacro" />
-  <xacro:include filename="$(find jackal_velodyne_vlp16_lidar_ros_nav_stack)/urdf/accessories/vlp16_mount.urdf.xacro" />
-  <xacro:include filename="$(find jackal_velodyne_vlp16_lidar_ros_nav_stack)/urdf/accessories/hdl32_mount.urdf.xacro" />
+  <xacro:include filename="$(find ros_stack_sim_jackal)/urdf/accessories/sick_lms1xx.urdf.xacro" />
+  <xacro:include filename="$(find ros_stack_sim_jackal)/urdf/accessories/sick_lms1xx_inverted_mount.urdf.xacro" />
+  <xacro:include filename="$(find ros_stack_sim_jackal)/urdf/accessories/sick_lms1xx_upright_mount.urdf.xacro" />
+  <xacro:include filename="$(find ros_stack_sim_jackal)/urdf/accessories/hokuyo_utm30.urdf.xacro" />
+  <xacro:include filename="$(find ros_stack_sim_jackal)/urdf/accessories/hokuyo_ust10.urdf.xacro" />
+  <xacro:include filename="$(find ros_stack_sim_jackal)/urdf/accessories/vlp16_mount.urdf.xacro" />
+  <xacro:include filename="$(find ros_stack_sim_jackal)/urdf/accessories/hdl32_mount.urdf.xacro" />
   <!--
     Add Microstrain IMU. By default the Jackal comes equipped with an IMU linked to "imu_link". These extra
@@ -195,6 +195,6 @@
     - smart7              :: Novatel Smart7
   -->
-  <xacro:include filename="$(find jackal_velodyne_vlp16_lidar_ros_nav_stack)/urdf/accessories/novatel_smart6.urdf.xacro" />
-  <xacro:include filename="$(find jackal_velodyne_vlp16_lidar_ros_nav_stack)/urdf/accessories/novatel_smart7.urdf.xacro" />
+  <xacro:include filename="$(find ros_stack_sim_jackal)/urdf/accessories/novatel_smart6.urdf.xacro" />
+  <xacro:include filename="$(find ros_stack_sim_jackal)/urdf/accessories/novatel_smart7.urdf.xacro" />
   <xacro:if value="$(optenv JACKAL_NAVSAT 0)">
     <xacro:property name="mount" value="$(optenv JACKAL_NAVSAT_MOUNT rear)" />
@@ -257,5 +257,5 @@
   -->
   <!-- Common camera mounts and accessory URDFs. -->
-  <xacro:include filename="$(find jackal_velodyne_vlp16_lidar_ros_nav_stack)/urdf/accessories/camera_mount.urdf.xacro" />
+  <xacro:include filename="$(find ros_stack_sim_jackal)/urdf/accessories/camera_mount.urdf.xacro" />
   <xacro:include filename="$(find pointgrey_camera_description)/urdf/pointgrey_flea3.urdf.xacro" />
   <!-- If enabled, generate the flea3 camera payload with a tilt of 30 degrees. -->
@@ -302,5 +302,5 @@
     </xacro:unless>
   </xacro:if>
-  <xacro:include filename="$(find jackal_velodyne_vlp16_lidar_ros_nav_stack)/urdf/accessories/stereo_camera_mount.urdf.xacro" />
+  <xacro:include filename="$(find ros_stack_sim_jackal)/urdf/accessories/stereo_camera_mount.urdf.xacro" />
   <!-- If enabled, generates a pair of flea3 cameras for stereo vision with a tilt of 30 degrees. -->
   <!-- Disabled temporarily due to metapackage issue. -->
@@ -396,5 +396,5 @@
   <!-- Fender Accessories -->
   <xacro:if value="$(optenv JACKAL_FRONT_ACCESSORY_FENDER 0)">
-    <xacro:include filename="$(find jackal_velodyne_vlp16_lidar_ros_nav_stack)/urdf/accessories/hokuyo_ust10.urdf.xacro" />
+    <xacro:include filename="$(find ros_stack_sim_jackal)/urdf/accessories/hokuyo_ust10.urdf.xacro" />
     <xacro:if value="$(optenv JACKAL_FRONT_FENDER_UST10 0)">
       <xacro:hokuyo_ust10_mount
@@ -425,5 +425,5 @@
       <visual>
         <geometry>
-          <mesh filename="package://jackal_velodyne_vlp16_lidar_ros_nav_stack/meshes/wibotic_bumper.stl" />
+          <mesh filename="package://ros_stack_sim_jackal/meshes/wibotic_bumper.stl" />
         </geometry>
         <material name="dark_grey" />
@@ -447,5 +447,5 @@
         <origin xyz="0 0 0" rpy="0 0 0"/>
         <geometry>
-          <mesh filename="package://jackal_velodyne_vlp16_lidar_ros_nav_stack/meshes/ark_enclosure.stl"/>
+          <mesh filename="package://ros_stack_sim_jackal/meshes/ark_enclosure.stl"/>
         </geometry>
         <material name="dark_grey" />

File: urdf/jackal.urdf.xacro (robot description, xacro)
@@ -22,5 +22,5 @@
         <origin xyz="0 0 0" rpy="${PI/2} 0 0"/>
         <geometry>
-          <mesh filename="package://jackal_velodyne_vlp16_lidar_ros_nav_stack/meshes/jackal-wheel.dae"/>
+          <mesh filename="package://ros_stack_sim_jackal/meshes/jackal-wheel.dae"/>
         </geometry>
         <material name="black" />
@@ -85,5 +85,5 @@
       <origin xyz="0 0 ${footprint_vertical_offset}" rpy="${PI/2} 0 ${PI/2}"/>
       <geometry>
-        <mesh filename="package://jackal_velodyne_vlp16_lidar_ros_nav_stack/meshes/jackal-base.dae"/>
+        <mesh filename="package://ros_stack_sim_jackal/meshes/jackal-base.dae"/>
       </geometry>
       <material name="dark_grey" />
@@ -110,5 +110,5 @@
       <origin xyz="0 0 ${footprint_vertical_offset}" rpy="${PI/2} 0 ${PI/2}"/>
       <geometry>
-        <mesh filename="package://jackal_velodyne_vlp16_lidar_ros_nav_stack/meshes/jackal-fenders.dae"/>
+        <mesh filename="package://ros_stack_sim_jackal/meshes/jackal-fenders.dae"/>
       </geometry>
       <material name="yellow" />
@@ -168,9 +168,9 @@
   </joint>
   <!-- Bring in simulation data for Gazebo. -->
-  <xacro:include filename="$(find jackal_velodyne_vlp16_lidar_ros_nav_stack)/urdf/jackal.gazebo" />
+  <xacro:include filename="$(find ros_stack_sim_jackal)/urdf/jackal.gazebo" />
   <!-- Optional standard accessories, including their simulation data. The rendering
        of these into the final description is controlled by optenv variables, which
        default each one to off.-->
-  <xacro:include filename="$(find jackal_velodyne_vlp16_lidar_ros_nav_stack)/urdf/accessories.urdf.xacro" />
+  <xacro:include filename="$(find ros_stack_sim_jackal)/urdf/accessories.urdf.xacro" />
   <!-- Optional custom includes. -->
   <xacro:if value="$(optenv JACKAL_URDF_EXTRAS 0)">
